Commit message: Implemented new nodes for manipulation, changed the package name to unitree_g1_dex3_stack. TODO: launch files and rviz config.

File: robots/g1_description/g1_29dof_with_hand_rev_1_0.urdf (robot description, URDF)
Before this commit: robot g1_29dof_lock_waist_with_hand_rev_1_0, 53 links, 52 joints
Joints:
- joint waist_pitch_joint: type fixed -> revolute
- joint waist_roll_joint: type fixed -> revolute
