Commit message: Lots of bug fixes, compilation issues and runtime launch file issues, planner.launch.py and perception.launch.py is still not ready.

File: robots/g1_description/g1_29dof_lock_waist_with_hand_rev_1_0.urdf (robot description, URDF)
Before this commit: robot g1_29dof_lock_waist_with_hand_rev_1_0, 53 links, 52 joints
Links:
- added link base_link
Joints:
- added joint base_to_pelvis: type fixed, parent base_link, child pelvis, origin xyz=0 0 0 rpy=0 0 0

Commit message: Updated urdf mesh paths

File: robots/g1_description/g1_29dof_lock_waist_with_hand_rev_1_0.urdf (robot description, URDF)
Before this commit: robot g1_29dof_lock_waist_with_hand_rev_1_0, 54 links, 53 joints
Links:
- link left_ankle_pitch_link: geometry collision mesh filename=package://unitree_g1_dex3_stack/robots/g1_description/meshe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; visual mesh filename=package://unitree_g1_dex3_stack/robots/g1_description/meshe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
- link left_ankle_roll_link: geometry collision sphere radius=0.005; collision sphere radius=0.005
- link left_elbow_link: geometry collision mesh filename=package://unitree_g1_dex3_stack/robots/g1_description/meshe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; visual mesh filename=package://unitree_g1_dex3_stack/robots/g1_description/meshe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
- link left_hip_pitch_link: geometry collision mesh filename=package://unitree_g1_dex3_stack/robots/g1_description/meshe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; visual mesh filename=package://unitree_g1_dex3_stack/robots/g1_description/meshe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
- link left_hip_roll_link: geometry collision mesh filename=package://unitree_g1_dex3_stack/robots/g1_description/meshe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; visual mesh filename=package://unitree_g1_dex3_stack/robots/g1_description/meshe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
- link left_hip_yaw_link: geometry collision mesh filename=package://unitree_g1_dex3_stack/robots/g1_description/meshe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; visual mesh filename=package://unitree_g1_dex3_stack/robots/g1_description/meshe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
- link left_knee_link: geometry collision mesh filename=package://unitree_g1_dex3_stack/robots/g1_description/meshe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; visual mesh filename=package://unitree_g1_dex3_stack/robots/g1_description/meshe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
- link left_shoulder_pitch_link: geometry collision cylinder length=0.05 radius=0.03; visual mesh filename=package://unitree_g1_dex3_stack/robots/g1_description/meshe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
- link left_shoulder_roll_link: geometry collision cylinder length=0.03 radius=0.03; visual mesh filename=package://unitree_g1_dex3_stack/robots/g1_description/meshe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
- link left_shoulder_yaw_link: geometry collision mesh filename=package://unitree_g1_dex3_stack/robots/g1_description/meshe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; visual mesh filename=package://unitree_g1_dex3_stack/robots/g1_description/meshe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
- link left_wrist_pitch_link: geometry collision mesh filename=package://unitree_g1_dex3_stack/robots/g1_description/meshe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; visual mesh filename=package://unitree_g1_dex3_stack/robots/g1_description/meshe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
- link left_wrist_roll_link: geometry collision mesh filename=package://unitree_g1_dex3_stack/robots/g1_description/meshe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; visual mesh filename=package://unitree_g1_dex3_stack/robots/g1_description/meshe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
- link left_wrist_yaw_link: geometry collision mesh filename=package://unitree_g1_dex3_stack/robots/g1_description/meshe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; visual mesh filename=package://unitree_g1_dex3_stack/robots/g1_description/meshe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
- link pelvis: geometry visual mesh filename=package://unitree_g1_dex3_stack/robots/g1_description/meshe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
- link pelvis_contour_link: geometry collision mesh filename=package://unitree_g1_dex3_stack/robots/g1_description/meshe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; visual mesh filename=package://unitree_g1_dex3_stack/robots/g1_description/meshe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
- link right_ankle_pitch_link: geometry collision mesh filename=package://unitree_g1_dex3_stack/robots/g1_description/meshe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; visual mesh filename=package://unitree_g1_dex3_stack/robots/g1_description/meshe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
- link right_ankle_roll_link: geometry collision sphere radius=0.005; collision sphere radius=0.005
- link right_elbow_link: geometry collision mesh filename=package://unitree_g1_dex3_stack/robots/g1_description/meshe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; visual mesh filename=package://unitree_g1_dex3_stack/robots/g1_description/meshe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
- link right_hip_pitch_link: geometry collision mesh filename=package://unitree_g1_dex3_stack/robots/g1_description/meshe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; visual mesh filename=package://unitree_g1_dex3_stack/robots/g1_description/meshe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
- link right_hip_roll_link: geometry collision mesh filename=package://unitree_g1_dex3_stack/robots/g1_description/meshe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; visual mesh filename=package://unitree_g1_dex3_stack/robots/g1_description/meshe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
- link right_hip_yaw_link: geometry collision mesh filename=package://unitree_g1_dex3_stack/robots/g1_description/meshe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; visual mesh filename=package://unitree_g1_dex3_stack/robots/g1_description/meshe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
- link right_knee_link: geometry collision mesh filename=package://unitree_g1_dex3_stack/robots/g1_description/meshe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; visual mesh filename=package://unitree_g1_dex3_stack/robots/g1_description/meshe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
- link right_shoulder_pitch_link: geometry collision cylinder length=0.05 radius=0.03; visual mesh filename=package://unitree_g1_dex3_stack/robots/g1_description/meshe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
- link right_shoulder_roll_link: geometry collision cylinder length=0.03 radius=0.03; visual mesh filename=package://unitree_g1_dex3_stack/robots/g1_description/meshe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
- link right_shoulder_yaw_link: geometry collision mesh filename=package://unitree_g1_dex3_stack/robots/g1_description/meshe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; visual mesh filename=package://unitree_g1_dex3_stack/robots/g1_description/meshe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
- link right_wrist_pitch_link: geometry collision mesh filename=package://unitree_g1_dex3_stack/robots/g1_description/meshe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; visual mesh filename=package://unitree_g1_dex3_stack/robots/g1_description/meshe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
- link right_wrist_roll_link: geometry collision mesh filename=package://unitree_g1_dex3_stack/robots/g1_description/meshe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; visual mesh filename=package://unitree_g1_dex3_stack/robots/g1_description/meshe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
- link right_wrist_yaw_link: geometry collision mesh filename=package://unitree_g1_dex3_stack/robots/g1_description/meshe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; visual mesh filename=package://unitree_g1_dex3_stack/robots/g1_description/meshe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
- link torso_link: geometry collision mesh filename=package://unitree_g1_dex3_stack/robots/g1_description/meshe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; visual mesh filename=package://unitree_g1_dex3_stack/robots/g1_description/meshe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
- link waist_roll_link: geometry visual mesh filename=package://unitree_g1_dex3_stack/robots/g1_description/meshe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
- link waist_yaw_link: geometry visual mesh filename=package://unitree_g1_dex3_stack/robots/g1_description/meshe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

Commit message: fix

File: robots/g1_description/g1_29dof_lock_waist_with_hand_rev_1_0.urdf (robot description, URDF)
Before this commit: robot g1_29dof_lock_waist_with_hand_rev_1_0, 54 links, 53 joints
Links:
- link head_link: geometry collision mesh filename=package://unitree_g1_dex3_stack/robots/g1_description/meshe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; visual mesh filename=package://unitree_g1_dex3_stack/robots/g1_description/meshe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
- link left_hand_index_0_link: geometry collision mesh filename=package://unitree_g1_dex3_stack/robots/g1_description/meshe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; visual mesh filename=package://unitree_g1_dex3_stack/robots/g1_description/meshe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
- link left_hand_index_1_link: geometry collision mesh filename=package://unitree_g1_dex3_stack/robots/g1_description/meshe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; visual mesh filename=package://unitree_g1_dex3_stack/robots/g1_description/meshe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
- link left_hand_middle_0_link: geometry collision mesh filename=package://unitree_g1_dex3_stack/robots/g1_description/meshe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; visual mesh filename=package://unitree_g1_dex3_stack/robots/g1_description/meshe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
- link left_hand_middle_1_link: geometry collision mesh filename=package://unitree_g1_dex3_stack/robots/g1_description/meshe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; visual mesh filename=package://unitree_g1_dex3_stack/robots/g1_description/meshe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
- link left_hand_palm_link: geometry collision mesh filename=package://unitree_g1_dex3_stack/robots/g1_description/meshe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; visual mesh filename=package://unitree_g1_dex3_stack/robots/g1_description/meshe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
- link left_hand_thumb_0_link: geometry collision mesh filename=package://unitree_g1_dex3_stack/robots/g1_description/meshe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; visual mesh filename=package://unitree_g1_dex3_stack/robots/g1_description/meshe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
- link left_hand_thumb_1_link: geometry collision box size=0.02 0.03 0.02; visual mesh filename=package://unitree_g1_dex3_stack/robots/g1_description/meshe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
- link left_hand_thumb_2_link: geometry collision mesh filename=package://unitree_g1_dex3_stack/robots/g1_description/meshe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; visual mesh filename=package://unitree_g1_dex3_stack/robots/g1_description/meshe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
- link logo_link: geometry collision mesh filename=package://unitree_g1_dex3_stack/robots/g1_description/meshe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; visual mesh filename=package://unitree_g1_dex3_stack/robots/g1_description/meshe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
- link right_hand_index_0_link: geometry collision mesh filename=package://unitree_g1_dex3_stack/robots/g1_description/meshe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; visual mesh filename=package://unitree_g1_dex3_stack/robots/g1_description/meshe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
- link right_hand_index_1_link: geometry collision mesh filename=package://unitree_g1_dex3_stack/robots/g1_description/meshe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; visual mesh filename=package://unitree_g1_dex3_stack/robots/g1_description/meshe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
- link right_hand_middle_0_link: geometry collision mesh filename=package://unitree_g1_dex3_stack/robots/g1_description/meshe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; visual mesh filename=package://unitree_g1_dex3_stack/robots/g1_description/meshe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
- link right_hand_middle_1_link: geometry collision mesh filename=package://unitree_g1_dex3_stack/robots/g1_description/meshe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; visual mesh filename=package://unitree_g1_dex3_stack/robots/g1_description/meshe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
- link right_hand_palm_link: geometry collision mesh filename=package://unitree_g1_dex3_stack/robots/g1_description/meshe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; visual mesh filename=package://unitree_g1_dex3_stack/robots/g1_description/meshe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
- link right_hand_thumb_0_link: geometry collision mesh filename=package://unitree_g1_dex3_stack/robots/g1_description/meshe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; visual mesh filename=package://unitree_g1_dex3_stack/robots/g1_description/meshe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
- link right_hand_thumb_1_link: geometry collision box size=0.02 0.03 0.02; visual mesh filename=package://unitree_g1_dex3_stack/robots/g1_description/meshe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
- link right_hand_thumb_2_link: geometry collision mesh filename=package://unitree_g1_dex3_stack/robots/g1_description/meshe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; visual mesh filename=package://unitree_g1_dex3_stack/robots/g1_description/meshe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

Commit message: Fixed G1 Locked Waist URDF with primitive collision geometries.

File: robots/g1_description/g1_29dof_lock_waist_with_hand_rev_1_0.urdf (robot description, URDF)
Before this commit: robot g1_29dof_lock_waist_with_hand_rev_1_0, 54 links, 53 joints
Links:
- link head_link: geometry collision cylinder length=0.2058 radius=0.0798; visual mesh filename=package://unitree_g1_dex3_stack/robots/g1_description/meshe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
- link left_ankle_pitch_link: geometry collision box size=0.0360 0.0130 0.0374; visual mesh filename=package://unitree_g1_dex3_stack/robots/g1_description/meshe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
- link left_elbow_link: geometry collision box size=0.1298 0.0660 0.0752; visual mesh filename=package://unitree_g1_dex3_stack/robots/g1_description/meshe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
- link left_hand_index_0_link: geometry collision box size=0.0618 0.0273 0.0257; visual mesh filename=package://unitree_g1_dex3_stack/robots/g1_description/meshe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
- link left_hand_index_1_link: geometry collision box size=0.0590 0.0177 0.0260; visual mesh filename=package://unitree_g1_dex3_stack/robots/g1_description/meshe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
- link left_hand_middle_0_link: geometry collision box size=0.0618 0.0273 0.0257; visual mesh filename=package://unitree_g1_dex3_stack/robots/g1_description/meshe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
- link left_hand_middle_1_link: geometry collision box size=0.0590 0.0177 0.0260; visual mesh filename=package://unitree_g1_dex3_stack/robots/g1_description/meshe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
- link left_hand_palm_link: geometry collision box size=0.0867 0.0417 0.0878; visual mesh filename=package://unitree_g1_dex3_stack/robots/g1_description/meshe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
- link left_hand_thumb_0_link: geometry collision box size=0.0216 0.0283 0.0190; visual mesh filename=package://unitree_g1_dex3_stack/robots/g1_description/meshe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
- link left_hand_thumb_2_link: geometry collision box size=0.0177 0.0590 0.0260; visual mesh filename=package://unitree_g1_dex3_stack/robots/g1_description/meshe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
- link left_hip_pitch_link: geometry collision box size=0.0826 0.0988 0.1172; visual mesh filename=package://unitree_g1_dex3_stack/robots/g1_description/meshe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
- link left_hip_roll_link: geometry collision box size=0.1065 0.0979 0.1706; visual mesh filename=package://unitree_g1_dex3_stack/robots/g1_description/meshe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
- link left_hip_yaw_link: geometry collision box size=0.1796 0.0887 0.2262; visual mesh filename=package://unitree_g1_dex3_stack/robots/g1_description/meshe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
- link left_knee_link: geometry collision box size=0.1038 0.0717 0.3551; visual mesh filename=package://unitree_g1_dex3_stack/robots/g1_description/meshe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
- link left_shoulder_yaw_link: geometry collision box size=0.0812 0.0745 0.1453; visual mesh filename=package://unitree_g1_dex3_stack/robots/g1_description/meshe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
- link left_wrist_pitch_link: geometry collision box size=0.1030 0.0570 0.0570; visual mesh filename=package://unitree_g1_dex3_stack/robots/g1_description/meshe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
- link left_wrist_roll_link: geometry collision cylinder length=0.0582 radius=0.0310; visual mesh filename=package://unitree_g1_dex3_stack/robots/g1_description/meshe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
- link left_wrist_yaw_link: geometry collision box size=0.0595 0.0539 0.0605; visual mesh filename=package://unitree_g1_dex3_stack/robots/g1_description/meshe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
- link logo_link: geometry collision box size=0.1494 0.1493 0.0292; visual mesh filename=package://unitree_g1_dex3_stack/robots/g1_description/meshe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
- link pelvis_contour_link: geometry collision box size=0.1196 0.1355 0.1242; visual mesh filename=package://unitree_g1_dex3_stack/robots/g1_description/meshe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
- link right_ankle_pitch_link: geometry collision box size=0.0360 0.0130 0.0374; visual mesh filename=package://unitree_g1_dex3_stack/robots/g1_description/meshe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
- link right_elbow_link: geometry collision box size=0.1298 0.0660 0.0752; visual mesh filename=package://unitree_g1_dex3_stack/robots/g1_description/meshe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
- link right_hand_index_0_link: geometry collision box size=0.0618 0.0273 0.0257; visual mesh filename=package://unitree_g1_dex3_stack/robots/g1_description/meshe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
- link right_hand_index_1_link: geometry collision box size=0.0590 0.0177 0.0260; visual mesh filename=package://unitree_g1_dex3_stack/robots/g1_description/meshe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
- link right_hand_middle_0_link: geometry collision box size=0.0618 0.0273 0.0257; visual mesh filename=package://unitree_g1_dex3_stack/robots/g1_description/meshe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
- link right_hand_middle_1_link: geometry collision box size=0.0590 0.0177 0.0260; visual mesh filename=package://unitree_g1_dex3_stack/robots/g1_description/meshe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
- link right_hand_palm_link: geometry collision box size=0.0867 0.0417 0.0878; visual mesh filename=package://unitree_g1_dex3_stack/robots/g1_description/meshe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
- link right_hand_thumb_0_link: geometry collision box size=0.0216 0.0283 0.0190; visual mesh filename=package://unitree_g1_dex3_stack/robots/g1_description/meshe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
- link right_hand_thumb_2_link: geometry collision box size=0.0177 0.0590 0.0260; visual mesh filename=package://unitree_g1_dex3_stack/robots/g1_description/meshe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
- link right_hip_pitch_link: geometry collision box size=0.0826 0.0988 0.1172; visual mesh filename=package://unitree_g1_dex3_stack/robots/g1_description/meshe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
- link right_hip_roll_link: geometry collision box size=0.1065 0.0979 0.1706; visual mesh filename=package://unitree_g1_dex3_stack/robots/g1_description/meshe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
- link right_hip_yaw_link: geometry collision box size=0.1796 0.0887 0.2262; visual mesh filename=package://unitree_g1_dex3_stack/robots/g1_description/meshe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
- link right_knee_link: geometry collision box size=0.1038 0.0717 0.3551; visual mesh filename=package://unitree_g1_dex3_stack/robots/g1_description/meshe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
- link right_shoulder_yaw_link: geometry collision box size=0.0812 0.0745 0.1453; visual mesh filename=package://unitree_g1_dex3_stack/robots/g1_description/meshe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
- link right_wrist_pitch_link: geometry collision box size=0.1030 0.0570 0.0570; visual mesh filename=package://unitree_g1_dex3_stack/robots/g1_description/meshe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
- link right_wrist_roll_link: geometry collision cylinder length=0.0582 radius=0.0310; visual mesh filename=package://unitree_g1_dex3_stack/robots/g1_description/meshe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
- link right_wrist_yaw_link: geometry collision box size=0.0595 0.0539 0.0605; visual mesh filename=package://unitree_g1_dex3_stack/robots/g1_description/meshe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
- link torso_link: geometry collision box size=0.1503 0.1954 0.3205; visual mesh filename=package://unitree_g1_dex3_stack/robots/g1_description/meshe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
